Commit message: 真实抓取版本

File: src/aubo_description/urdf/aubo_i5H.urdf (robot description, URDF)
Before this commit: robot aubo_i5H, 11 links, 10 joints
Joints:
- joint afinger1_joint: type prismatic -> fixed
- joint afinger2_joint: type prismatic -> fixed

File: src/aubo_i5h_moveit1/config/aubo_i5H.ros2_control.xacro (robot description, xacro)
@@ -56,4 +56,7 @@
                 <state_interface name="velocity"/>
             </joint>
+            <joint name="afinger2_joint">
+                <state_interface name="position"/>
+            </joint>
         </ros2_control>
     </xacro:macro>
